File: MP2636-Single-Cell-BMS/MP2636-Single-Cell-BMS.sch (EAGLE design)
At the start: 43 parts, among them U1 MP2636GR-P

Commit message: Updated names and values
Parts:
- removed C10: NC, Capacitor:C_CHIP-0805(2012-METRIC)
- removed C11, C12: 22uf, Capacitor:C_CHIP-0805(2012-METRIC)
- removed R13, R14, R15: 2K, Resistor:R-US_CHIP-0805(2012-METRIC)
- removed R17: 10K, Resistor:R-US_CHIP-0805(2012-METRIC)
- added CBATT, CIN, CSYS: 22uf, Capacitor:C_CHIP-0805(2012-METRIC)
- added F, JP11, JP18: SYS, Connector:PINHD-1X1
- added JP10: AGND, Connector:PINHD-1X1
- added JP12: IB, Connector:PINHD-1X1
- added JP13, JP14: BATT, Connector:PINHD-1X1
- added JP15: NTC, Connector:PINHD-1X1
- added JP16: SW, Connector:PINHD-1X1
- added JP17, JP6: PGND, Connector:PINHD-1X1
- added JP4, JP9: VIN, Connector:PINHD-1X1
- added JP7: PWIN, Connector:PINHD-1X1
- added JP8: VCC, Connector:PINHD-1X1
- added RH: 15K 1%, Resistor:R-US_CHIP-0805(2012-METRIC)
- added RL: 5.1K, Resistor:R-US_CHIP-0805(2012-METRIC)
- added RS1: 20m, Resistor:R-US_CHIP-0805(2012-METRIC)
- added RT2: 10K, Resistor:R-US_CHIP-0805(2012-METRIC)
- C1: value 100nf -> 1uf
- C3: value 1uf -> 22uf
- C4: value 22uf -> 100nf
- C7: value (none) -> 22uf
- C8: value 22uf -> (none)
- C9: value 22uf -> NC
- R1: value 10K -> 31.6K
- R10: value 10K -> 2K
- R11: value 1K -> 2K
- R12: value 20m -> 1K
- R3: value 10K -> 23.7K 1%
- R4: value 15K -> 5.1K
- R5, R7: value 5.1K -> 10K
- R6: value 23.7K -> 10K
- R9: value 31.6K -> 2K
- ROLIM: value 37.4K -> 37.4K 1%
- renumbered C13 to CTMR, J1 to JP1, J2 to JP2, J3 to JP3, J4 to JP5, R16 to RT1, R18 to RILIM, R19 to RISET, R20 to ROLIM, R8 to RT
Connections:
- net N$19 renamed HIGH
- removed net N$13: C11.1, C12.1
- net AGND: now also JP10.1, R2.2, R4.1, RL.1, RT2.1; no longer R10.2, R17.1, R5.1, R7.1
- net DGND: now also C1.1, C4.2, C7.1, C9.2, CBATT.1, CIN.1, CSYS.1, JP17.1, JP6.1; no longer C1.2, C10.2, C4.1, C8.1, C9.1
- net IB: now also C9.1, JP12.1, R12.2; no longer C10.1, R11.2
- net N$1: now also R12.1; no longer R11.1
- net N$10: now also C8.2, R1.2, R2.1; no longer C7.2, R10.1, R9.2
- net N$12: now also RS1.1; no longer R12.1
- net N$15: now also R9.1; no longer R13.1
- net N$16: now also R10.1; no longer R14.1
- net N$17: now also R11.1; no longer R15.1
- net N$18: now also R10.2, R11.2, R9.2; no longer R13.2, R14.2, R15.2
- net N$2: now also R5.2; no longer R1.2
- net N$6: now also R6.2; no longer R2.2
- net N$7: now also R7.2; no longer R3.2
- net N$8: now also RH.1, RL.2; no longer R4.1, R5.2
- net NTC: now also JP15.1, RT2.2; no longer R17.2
- net PWIN: now also JP7.1, R3.1, R4.2; no longer R6.1, R7.2
- net SW: now also JP16.1
- net SYS: now also C2.2, C7.2, C8.1, CSYS.2, F.1, JP11.1, JP18.1, R1.1; no longer C5.2, C7.1, C8.2, C9.2, R9.1
- net VBATT: now also C3.2, CBATT.2, JP13.1, JP14.1, RS1.2; no longer C11.2, C12.2, R12.2
- net VCC: now also C4.1, JP8.1, R5.1, R6.1, R7.1; no longer C1.1, R1.1, R2.1, R3.1
- net VIN: now also C1.2, C5.2, CIN.2, JP4.1, JP9.1, R3.2, RH.2; no longer C2.2, C3.2, C4.2, R4.2, R6.2
Other:
- moved on the sheet: C1, C2, C3, C4, C5, C7, C8, C9, R1, R10, R11, R12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
